File: new_fretboard_rev4/new_fretboard_rev4/new_fretboard_rev4.kicad_pcb (KiCad board)
At the start: 4 copper layers, 585 x 79 mm, 47 parts, among them CN1 Header 1x6, CN2 Header 1x6, J1 JMP, J2 JMP, J4 JMP, J8 JMP, U1 LX3302AQPW_TSSOP-14, U2 LX3302AQPW_TSSOP-14

Commit message: possibly correct net names for coils
Connections:
- J4 pad 1: Net-(J4-Pad1) -> /OSC_CW_A
Routing:
- net Net-(J4-Pad1): track 2184.3 -> 0.00 mm, vias 1 -> 0
- net /OSC_CW_A: track 0.00 -> 2184.3 mm, vias 0 -> 1
- net /COS_A: track 4225.7 -> 2104.1 mm, vias 39 -> 36
- net /COS_B: track 0.00 -> 2116.2 mm, vias 0 -> 43
- net Net-(U2-IO4): track 16.1 -> 0.00 mm
- net Net-(U2-IO3): track 14.5 -> 0.00 mm
- net Net-(U1-IO4): track 12.7 -> 0.00 mm
- net Net-(U2-IO1): track 11.2 -> 0.00 mm
- net Net-(U1-IO3): track 10.9 -> 0.00 mm
- net VDD1: track 10.8 -> 0.00 mm
- net /SUB: track 8.88 -> 0.00 mm
- net /SIN_A: track 2083.0 -> 2074.2 mm, vias 38 -> 36
- net GND1: track 26.8 -> 18.7 mm
- net VIN1: track 7.91 -> 0.00 mm
- net Net-(U1-IO1): track 7.91 -> 0.00 mm
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