File: new_fretboard_rev4/new_fretboard_rev4/new_fretboard_rev4.kicad_pcb (KiCad board)
At the start: 4 copper layers, 585 x 79 mm, 48 parts, among them J1 Conn_01x06, J2 Conn_01x06, U1 LX3302AQPW_TSSOP-14, U2 LX3302AQPW_TSSOP-14

Commit message: top layer routed, starting bottom layer
Parts:
- moved L2 3.34 mm to (32.3, 131.8)
- moved L6 3.09 mm to (31.8, 130.8)
- moved L1 3.09 mm to (32.0, 132.3), turned to -90 degrees
- moved L5 3.08 mm to (32.0, 132.8)
- moved L3 0.44 mm to (46.5, 132.1)
Routing:
- net /OSC_CCW_A: track 2182.3 -> 4378.8 mm, vias 0 -> 5
- net /OSC_CW_B: track 0.00 -> 2181.6 mm
- net /OSC_CCW_B: track 2180.5 -> 0.00 mm
- net /OSC_CW_A: track 4370.7 -> 2198.1 mm, vias 0 -> 2
- net GND1: track 21.1 -> 53.7 mm, vias 6 -> 10
- net /SIN_A: track 2054.8 -> 2077.3 mm, vias 36 -> 38
- net /COS_A: track 2100.4 -> 2118.1 mm, vias 36 -> 38
- net /IO4_A: track 0.00 -> 14.3 mm, vias 0 -> 1
- net /IO3_A: track 0.00 -> 12.0 mm, vias 0 -> 1
- net /IO2_A: track 4.69 -> 15.1 mm, vias 0 -> 2
- net /IO1_A: track 6.98 -> 16.9 mm
- net /OSC_RTN_A: track 0.00 -> 7.22 mm, vias 0 -> 2
- net /VIN_A: track 2.32 -> 8.09 mm, vias 0 -> 1
