File: new_fretboard_rev4/new_fretboard_rev4/new_fretboard_rev4.kicad_sch (KiCad schematic)
At the start: 48 parts, among them J1 Conn_01x06, J2 Conn_01x05, U1 LX3302AQPW_TSSOP-14, U2 LX3302AQPW_TSSOP-14

Commit message: channels are done, working on microcontroller, daisy, and power junctions. getting heirarchical pin stuff sorted.
Connections:
- net IO2_A_FILT renamed SENTOUT_OUT
- net VIN_A renamed VIN_IN
Changed lines of the file:
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@@
+		)
+	)
+	(hierarchical_label "VIN_IN"
+		(shape input)
+		(at 60.96 52.07 0)
+		(effects
+			(font
+				(size 1.27 1.27)
+			)
+			(justify left)
+		)
+	)
+	(hierarchical_label "SENTOUT_OUT"
+		(shape input)
+		(at 58.42 57.15 0)
+		(effects
+			(font
+				(size 1.27 1.27)
+			)
+			(justify left)
 		)
 	)

Commit message: power in schematic, about to route power and sent wires
Connections:
- net IO2_B_FILT renamed SENTOUT_OUT_B
- net SENTOUT_OUT renamed SENTOUT_OUT_A
- net VIN_B renamed VIN_IN_B
- net VIN_IN renamed VIN_IN_A
Changed lines of the file:
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@@
 		)
 	)
-	(hierarchical_label "VIN_IN"
+	(hierarchical_label "VIN_IN_A"
 		(shape input)
 		(at 60.96 52.07 0)
@@
 		)
 	)
-	(hierarchical_label "SENTOUT_OUT"
+	(hierarchical_label "SENTOUT_OUT_B"
 		(shape input)
+		(at 55.88 152.4 0)
+		(effects
+			(font
+				(size 1.27 1.27)
+			)
+			(justify left)
+		)
+	)
+	(hierarchical_label "SENTOUT_OUT_A"
+		(shape output)
 		(at 58.42 57.15 0)
 		(effects
 			(font
+				(size 1.27 1.27)
+			)
+			(justify left)
+		)
+	)
+	(hierarchical_label "VIN_IN_B"
+		(shape input)
+		(at 58.42 147.32 0)
+		(effects
+			(font
