File: new_fretboard_rev4/new_fretboard_rev6/new_fretboard_rev6.kicad_pcb (KiCad board)
At the start: 4 copper layers, 585 x 79 mm, 48 parts, among them J1 Conn_01x06, J2 Conn_01x06, U1 LX3302AQPW_TSSOP-14, U2 LX3302AQPW_TSSOP-14

Commit message: trying multichannel, reannotating
Parts:
- renumbered C16 to C15, C18 to C17, C5 to C6, L7 to L5, L8 to L6, R2 to R1, R4 to R3, R6 to R5
