File: new_fretboard_rev4/new_fretboard_rev6/new_fretboard_rev6.kicad_pcb (KiCad board)
At the start: 4 copper layers, 585 x 79 mm, 48 parts, among them J1 Conn_01x06, J2 Conn_01x06, U1 LX3302AQPW_TSSOP-14, U2 LX3302AQPW_TSSOP-14

Commit message: finished routing one channel. passes ERC. about to import second channel
Parts:
- moved L4 0.33 mm to (-201.1, 207.5)
- moved L2 0.22 mm to (-201.8, 208.2)
- renumbered J2 to J1, J1 to J2, L5 to L1, L1 to L2, L6 to L3, L2 to L4
Connections:
- net /COS_A renamed /ch1/COS_A
- net /COS_A_PRE_RES renamed /ch1/COS_A_PRE_RES
- net /COS_B renamed /ch1/COS_B
- net /COS_B_PRE_RES renamed /ch1/COS_B_PRE_RES
- net /IO1_A renamed /ch1/IO1_A
- net /IO1_B renamed /ch1/IO1_B
- net /IO2_A renamed /ch1/IO2_A
- net /IO2_A_FILT renamed /ch1/IO2_A_FILT
- net /IO2_B renamed /ch1/IO2_B
- net /IO2_B_FILT renamed /ch1/IO2_B_FILT
- net /IO3_A renamed /ch1/IO3_A
- net /IO3_B renamed /ch1/IO3_B
- net /IO4_A renamed /ch1/IO4_A
- net /IO4_B renamed /ch1/IO4_B
- net /OSC_CCW_A renamed /ch1/OSC_CCW_A
- net /OSC_CCW_B renamed /ch1/OSC_CCW_B
- net /OSC_CW_A renamed /ch1/OSC_CW_A
- net /OSC_CW_B renamed /ch1/OSC_CW_B
- net /OSC_RTN_A renamed /ch1/OSC_RTN_A
- net /OSC_RTN_B renamed /ch1/OSC_RTN_B
- net /SIN_A renamed /ch1/SIN_A
- net /SIN_A_PRE_RES renamed /ch1/SIN_A_PRE_RES
- net /SIN_B renamed /ch1/SIN_B
- net /SIN_B_PRE_RES renamed /ch1/SIN_B_PRE_RES
- net /SUB_A renamed /ch1/SUB_A
- net /SUB_B renamed /ch1/SUB_B
- net /VDD1_A renamed /ch1/VDD1_A
- net /VDD1_B renamed /ch1/VDD1_B
- net /VIN1_A renamed /ch1/VIN1_A
- net /VIN1_B renamed /ch1/VIN1_B
- net /VIN_A renamed /ch1/VIN_A
- net /VIN_B renamed /ch1/VIN_B
Routing:
- net /ch1/OSC_RTN_A: track 6.86 -> 7.62 mm
