File: new_fretboard_rev4/new_fretboard_rev6/new_fretboard_rev6.kicad_pcb (KiCad board)
At the start: 4 copper layers, 585 x 79 mm, 48 parts, among them J1 Conn_01x06, J2 Conn_01x06, U1 LX3302AQPW_TSSOP-14, U2 LX3302AQPW_TSSOP-14

Commit message: two channels done
Parts:
- added C301: 6.8nF, PCM_4ms_Capacitor:C_0603, B.Cu at (-220.1, 223.3)
- added C302: 6.8nF, PCM_4ms_Capacitor:C_0603, F.Cu at (-219.8, 219.5)
- added C303: 6.8nF, PCM_4ms_Capacitor:C_0603, B.Cu at (-220.6, 216.5)
- added C304: 6.8nF, PCM_4ms_Capacitor:C_0603, F.Cu at (-220.0, 226.3)
- added C305: 100nF, PCM_4ms_Capacitor:C_0603, B.Cu at (-218.9, 216.5)
- added C306: 100nF, PCM_4ms_Capacitor:C_0603, F.Cu at (-217.8, 226.4)
- added C307: 1000pF, PCM_4ms_Capacitor:C_0603, B.Cu at (-214.6, 215.5)
- added C308: 1000pF, PCM_4ms_Capacitor:C_0603, F.Cu at (-214.8, 226.4)
- added C309: 470nF, PCM_4ms_Capacitor:C_0603, B.Cu at (-211.0, 215.3)
- added C310: 470nF, PCM_4ms_Capacitor:C_0603, F.Cu at (-213.3, 226.4)
- added C311: 1uF, PCM_4ms_Capacitor:C_0603, B.Cu at (-208.8, 216.9)
- added C312: 1uF, PCM_4ms_Capacitor:C_0603, F.Cu at (-211.8, 226.4)
- added C313: 100nF, PCM_4ms_Capacitor:C_0603, B.Cu at (-217.5, 223.8)
- added C314: 100nF, PCM_4ms_Capacitor:C_0603, F.Cu at (-216.8, 219.5)
- added C315: 10pF, PCM_4ms_Capacitor:C_0603, B.Cu at (-210.9, 226.4)
- added C316: 10pF, PCM_4ms_Capacitor:C_0603, F.Cu at (-208.6, 216.8)
- added C317: 10pF, PCM_4ms_Capacitor:C_0603, B.Cu at (-212.4, 226.4)
- added C318: 10pF, PCM_4ms_Capacitor:C_0603, F.Cu at (-210.7, 215.2)
- added C319: 680PF, PCM_4ms_Capacitor:C_0603, B.Cu at (-215.4, 226.4)
- added C320: 680PF, PCM_4ms_Capacitor:C_0603, B.Cu at (-213.9, 226.4)
- added C321: 680PF, PCM_4ms_Capacitor:C_0603, F.Cu at (-217.6, 216.7)
- added C322: 680PF, PCM_4ms_Capacitor:C_0603, F.Cu at (-217.6, 215.1)
- added J301: Conn_01x06, Connector_PinHeader_2.54mm:PinHeader_1x05_P2.54mm_Vertical, F.Cu at (-226.7, 227.1)
- added J302: Conn_01x05, Connector_PinHeader_2.54mm:PinHeader_1x05_P2.54mm_Vertical, F.Cu at (-223.0, 226.9)
- added L301: PCB L, jumpers_custom:jumper_tiny, B.Cu at (-200.4, 219.5)
- added L302: PCB L, jumpers_custom:jumper_tiny, F.Cu at (-201.8, 222.4)
- added L303: PCB L, jumpers_custom:jumper_tiny, B.Cu at (-201.2, 219.2)
- added L304: PCB L, jumpers_custom:jumper_tiny, F.Cu at (-201.1, 221.8)
- added L305: PCB L, jumpers_custom:jumper_tiny, B.Cu at (-187.2, 222.5)
- added L306: PCB L, jumpers_custom:jumper_tiny, B.Cu at (-187.2, 222.3)
- added L307: PCB L, jumpers_custom:jumper_tiny, F.Cu at (-187.2, 222.0)
- added L308: PCB L, jumpers_custom:jumper_tiny, F.Cu at (-185.5, 221.8)
- added R301: 221R, PCM_4ms_Resistor:R_0603, B.Cu at (-220.5, 220.0)
- added R302: 221R, PCM_4ms_Resistor:R_0603, F.Cu at (-220.2, 222.8)
- added R303: 10k, PCM_4ms_Resistor:R_0603, B.Cu at (-217.1, 219.9)
- added R304: 10k, PCM_4ms_Resistor:R_0603, F.Cu at (-216.8, 222.8)
- added R305: 10k, PCM_4ms_Resistor:R_0603, B.Cu at (-218.7, 219.9)
- added R306: 10k, PCM_4ms_Resistor:R_0603, F.Cu at (-218.4, 222.8)
- added R307: 4.7R, PCM_4ms_Resistor:R_0603, B.Cu at (-217.2, 216.5)
- added R308: 4.7R, PCM_4ms_Resistor:R_0603, F.Cu at (-216.3, 226.4)
- added R309: 10R, PCM_4ms_Resistor:R_0603, B.Cu at (-208.8, 218.5)
- added R310: 10R, PCM_4ms_Resistor:R_0603, F.Cu at (-208.5, 223.0)
- added R311: 10R, PCM_4ms_Resistor:R_0603, B.Cu at (-208.9, 220.2)
- added R312: 10R, PCM_4ms_Resistor:R_0603, B.Cu at (-208.9, 222.0)
- added R313: 10R, PCM_4ms_Resistor:R_0603, F.Cu at (-208.6, 221.3)
- added R314: 10R, PCM_4ms_Resistor:R_0603, F.Cu at (-208.6, 219.5)
- added U301: LX3302AQPW_TSSOP-14, PCM_4ms_Package_SSOP:TSSOP-14_4.4x5mm_P0.65mm, B.Cu at (-213.3, 220.7)
- added U302: LX3302AQPW_TSSOP-14, PCM_4ms_Package_SSOP:TSSOP-14_4.4x5mm_P0.65mm, F.Cu at (-213.1, 220.6)
- J1: footprint Connector_PinHeader_2.54mm:PinHeader_1x06_P2.54mm_Vertical -> Connector_PinHeader_2.54mm:PinHeader_1x05_P2.54mm_Vertical
- J2: value Conn_01x06 -> Conn_01x05; footprint Connector_PinHeader_2.54mm:PinHeader_1x06_P2.54mm_Vertical -> Connector_PinHeader_2.54mm:PinHeader_1x05_P2.54mm_Vertical
- moved J2 41.3 mm to (-223.0, 241.2), turned to 180 degrees
- moved J1 41.2 mm to (-226.6, 241.4), turned to 180 degrees
- moved C11 30.6 mm to (-208.8, 231.3), turned to 180 degrees
- moved C16 30.5 mm to (-208.6, 231.2), turned to 180 degrees
- moved C13 30.4 mm to (-217.5, 238.1)
- moved C21 30.4 mm to (-217.6, 231.0), turned to 0 degrees
- moved C5 30.0 mm to (-218.8, 230.8)
- moved R7 30.0 mm to (-217.2, 230.8)
- moved C3 30.0 mm to (-220.6, 230.9)
- moved R1 30.0 mm to (-220.4, 234.3)
- moved C1 29.9 mm to (-220.1, 237.7)
- moved R3 29.9 mm to (-217.1, 234.2)
- moved R5 29.9 mm to (-218.7, 234.2)
- moved C7 29.1 mm to (-214.6, 229.9), turned to 0 degrees
- moved C9 29.0 mm to (-211.0, 229.6), turned to 180 degrees
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Connections:
- J1 pad 1: /ch1/IO4_B -> GND1
- J1 pad 2: /ch1/IO1_B -> /ch1/VIN_B
- J1 pad 3: /ch1/IO2_B_FILT -> /ch1/IO3_B
- J1 pad 4: /ch1/IO3_B -> /ch1/IO2_B_FILT
- J1 pad 5: /ch1/VIN_B -> /ch1/IO1_B
- J2 pad 1: /ch1/IO4_A -> GND1
- J2 pad 2: /ch1/IO1_A -> /ch1/VIN_A
- J2 pad 3: /ch1/IO2_A_FILT -> /ch1/IO3_A
- J2 pad 4: /ch1/IO3_A -> /ch1/IO2_A_FILT
- J2 pad 5: /ch1/VIN_A -> /ch1/IO1_A
- U1 pad 1: /ch1/IO4_B -> unconnected-(U1-IO4-Pad1)
- U2 pad 1: /ch1/IO4_A -> unconnected-(U2-IO4-Pad1)
Routing:
- net /ch2/OSC_CW_B: track 0.00 -> 2202.3 mm, vias 0 -> 3
- net /ch2/OSC_CCW_A: track 0.00 -> 2201.5 mm, vias 0 -> 5
- net /ch2/OSC_CW_A: track 0.00 -> 2199.6 mm, vias 0 -> 2
- net /ch2/OSC_CCW_B: track 0.00 -> 2195.6 mm, vias 0 -> 4
- net /ch2/COS_B: track 0.00 -> 2135.8 mm, vias 0 -> 44
- net /ch2/COS_A: track 0.00 -> 2117.9 mm, vias 0 -> 38
- net /ch2/SIN_B: track 0.00 -> 2098.1 mm, vias 0 -> 44
- net /ch2/SIN_A: track 0.00 -> 2077.7 mm, vias 0 -> 38
- net GND1: track 91.9 -> 180.5 mm, vias 20 -> 34
- net /ch2/IO1_B: track 0.00 -> 28.3 mm, vias 0 -> 2
- net /ch2/VIN_B: track 0.00 -> 21.3 mm, vias 0 -> 1
- net /ch2/VIN1_B: track 0.00 -> 20.9 mm
- net /ch2/IO1_A: track 0.00 -> 16.5 mm, vias 0 -> 2
- net /ch2/IO3_B: track 0.00 -> 16.4 mm, vias 0 -> 1
- net /ch2/VDD1_B: track 0.00 -> 16.1 mm, vias 0 -> 2
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